Commit message: + led

File: urdf/led.urdf (robot description, URDF)
Before this commit: robot m4k, 16 links, 15 joints
Links:
- removed link base_link
- removed link front_caster
- removed link front_wheel
- removed link left_wheel
- removed link rear_caster
- removed link rear_wheel
- removed link right_wheel
Joints:
- removed joint front_caster_joint
- removed joint front_wheel_joint
- removed joint led_joint
- removed joint left_wheel_joint
- removed joint rear_caster_joint
- removed joint rear_wheel_joint
- removed joint right_wheel_joint
