Commit message: +laser,ultrasonic

File: urdf/m4k.urdf (robot description, URDF)
Before this commit: robot m4k, 16 links, 15 joints
Links:
- added link laser; visual cylinder length=0.08 radius=0.035
- added link ultrasonic; visual box size=0.02 0.04 0.02
Joints:
- added joint hokuyo_joint: type fixed, parent base_link, child laser, origin xyz=0 0 0.29 rpy=0 0 0, axis 0 0 0
- added joint sonar_joint: type fixed, parent base_link, child ultrasonic, origin xyz=0.26 0 0.1
